File: CubeSat-Main/CubeSat_Main.kicad_sch (KiCad schematic)
At the start: 20 parts, among them J1 Conn_01x03_Pin, J2 Conn_01x08_Socket, U1 STM32F411CEU6 - BlackPill, U2 LORA E220-900T22D, U3 BNO055, U4 LM35-LP, U5 GPS_NEO6M

Commit message: minor changes in the design
Parts:
- renumbered D2 to D1, D3 to D2, D1 to D3
Connections:
- net LED_BLUE: now also R4.1, U1.4 (PC15); no longer R5.1, U1.3 (PC14)
- net LED_RED: now also R5.1, U1.3 (PC14); no longer R4.1, U1.4 (PC15)
Other:
- note added: "FAULT LED"
- note added: "STATUS LED"
- note removed: "ERROR STATUS"
- note removed: "OTHER STATUS"
Changed lines of the file:
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@@
 		)
 	)
-	(text "OTHER STATUS"
+	(text "FAULT LED"
 		(exclude_from_sim no)
 		(at 197.612 128.778 0)
@@
 		)
 	)
-	(text "ERROR STATUS"
+	(text "STATUS LED"
 		(exclude_from_sim no)
-		(at 170.18 128.778 0)
+		(at 171.704 129.032 0)
 		(effects
 			(font
@@
 		)
 	)
-	(global_label "LED_RED"
+	(global_label "LED_BLUE"
 		(shape input)
 		(at 123.19 133.35 0)
@@
 		)
 		(property "Intersheetrefs" "${INTERSHEET_REFS}"
-			(at 134.7549 133.35 0)
+			(at 135.8435 133.35 0)
 			(effects
 				(font
@@
 		)
 	)
-	(global_label "LED_BLUE"
+	(global_label "LED_RED"
 		(shape input)
 		(at 121.92 135.89 0)
@@
 		)
 		(property "Intersheetrefs" "${INTERSHEET_REFS}"
-			(at 134.5735 135.89 0)
+			(at 133.4849 135.89 0)
 			(effects
 				(font
@@
 		)
 	)
-	(global_label "LED_BLUE"
+	(global_label "LED_RED"
 		(shape input)
 		(at 196.85 134.62 0)
@@
 		)
 		(property "Intersheetrefs" "${INTERSHEET_REFS}"
-			(at 209.5035 134.62 0)
+			(at 208.4149 134.62 0)
 			(effects
 				(font
@@
 		)
 	)
-	(global_label "LED_RED"
+	(global_label "LED_BLUE"
 		(shape input)
 		(at 170.18 134.62 0)
@@
 		)
 		(property "Intersheetrefs" "${INTERSHEET_REFS}"
-			(at 181.7449 134.62 0)
+			(at 182.8335 134.62 0)
 			(effects
 				(font
@@
 		(dnp no)
 		(fields_autoplaced yes)
-		(property "Reference" "D3"
+		(property "Reference" "D2"
 			(at 196.85 150.1774 90)
 			(effects
@@
 			(project "CubesatMain"
 				(path "/efe2bccd-e118-4ad0-853a-c0e965c7d995"
-					(reference "D3")
+					(reference "D2")
 					(unit 1)
 				)
@@
 		(dnp no)
 		(fields_autoplaced yes)
-		(property "Reference" "D2"
+		(property "Reference" "D1"
 			(at 171.45 150.1774 90)
 			(effects
@@
 			(project ""
 				(path "/efe2bccd-e118-4ad0-853a-c0e965c7d995"
-					(reference "D2")
+					(reference "D1")
 					(unit 1)
 				)
@@
 		(dnp no)
 		(fields_autoplaced yes)
-		(property "Reference" "D1"
+		(property "Reference" "D3"
 			(at 270.51 106.9974 90)
 			(effects
@@
 			(project "CubesatMain"
 				(path "/efe2bccd-e118-4ad0-853a-c0e965c7d995"
-					(reference "D1")
+					(reference "D3")
 					(unit 1)
 				)
